File: boards/proto-half/proto-half.sch (KiCad schematic (older format))
At the start: 42 parts, among them J1 Conn_01x12, J10 Conn_01x12, J11 Conn_01x12, J12 Conn_01x12, J13 Conn_01x12, J14 Conn_01x12, J15 Conn_01x12, J16 Conn_01x12, J17 Conn_01x12, J18 Conn_01x12, J19 Conn_01x12, J2 Conn_01x12, J20 Conn_01x12, J21 Conn_01x12, J22 Conn_01x12, J23 Conn_01x12, J24 Conn_01x12, J25 Conn_01x12, J26 Conn_01x12, J27 Conn_01x12, J28 Conn_01x12, J29 Conn_01x12, J3 Conn_01x12, J30 Conn_01x12, J31 Conn_01x06, J32 Conn_01x06, J33 Conn_01x30, J34 Conn_01x30, J35 Conn_01x22, J36 Conn_01x22, J37 Conn_01x04_MountingPin, J38 Conn_01x04_MountingPin, J4 Conn_01x12, J5 Conn_01x12, J6 Conn_01x12, J7 Conn_01x12, J8 Conn_01x12, J9 Conn_01x12

Commit message: Start to fix the proto board connectors.
Half board is fixed, quarter board requires reducing the length of a couple
of the connectors, namely the power rails and the top-right proto line.
Parts:
- J37, J38: footprint Connector_JST:JST_SH_BM04B-SRSS-TB_1x04-1MP_P1.00mm_Vertical -> Connector_JST:JST_SH_SM04B-SRSS-TB_1x04-1MP_P1.00mm_Horizontal
Connections:
- net Q1-3v3: now also J3.10 (Pin_10), J3.11 (Pin_11), J3.12 (Pin_12), J3.8 (Pin_8), J3.9 (Pin_9); no longer J2.10 (Pin_10), J2.11 (Pin_11), J2.12 (Pin_12), J2.8 (Pin_8), J2.9 (Pin_9)
- net Q1-GND: now also J4.10 (Pin_10), J4.11 (Pin_11), J4.12 (Pin_12), J4.8 (Pin_8), J4.9 (Pin_9); no longer J1.10 (Pin_10), J1.11 (Pin_11), J1.12 (Pin_12), J1.8 (Pin_8), J1.9 (Pin_9)
- net Q1-SCL: now also J1.10 (Pin_10), J1.11 (Pin_11), J1.12 (Pin_12), J1.8 (Pin_8), J1.9 (Pin_9); no longer J4.10 (Pin_10), J4.11 (Pin_11), J4.12 (Pin_12), J4.8 (Pin_8), J4.9 (Pin_9)
- net Q1-SDA: now also J2.10 (Pin_10), J2.11 (Pin_11), J2.12 (Pin_12), J2.8 (Pin_8), J2.9 (Pin_9); no longer J3.10 (Pin_10), J3.11 (Pin_11), J3.12 (Pin_12), J3.8 (Pin_8), J3.9 (Pin_9)
- net Q2-3v3: now also J29.10 (Pin_10), J29.11 (Pin_11), J29.12 (Pin_12), J29.8 (Pin_8), J29.9 (Pin_9); no longer J28.10 (Pin_10), J28.11 (Pin_11), J28.12 (Pin_12), J28.8 (Pin_8), J28.9 (Pin_9)
- net Q2-GND: now also J30.10 (Pin_10), J30.11 (Pin_11), J30.12 (Pin_12), J30.8 (Pin_8), J30.9 (Pin_9); no longer J27.10 (Pin_10), J27.11 (Pin_11), J27.12 (Pin_12), J27.8 (Pin_8), J27.9 (Pin_9)
- net Q2-SCL: now also J27.10 (Pin_10), J27.11 (Pin_11), J27.12 (Pin_12), J27.8 (Pin_8), J27.9 (Pin_9); no longer J30.10 (Pin_10), J30.11 (Pin_11), J30.12 (Pin_12), J30.8 (Pin_8), J30.9 (Pin_9)
- net Q2-SDA: now also J28.10 (Pin_10), J28.11 (Pin_11), J28.12 (Pin_12), J28.8 (Pin_8), J28.9 (Pin_9); no longer J29.10 (Pin_10), J29.11 (Pin_11), J29.12 (Pin_12), J29.8 (Pin_8), J29.9 (Pin_9)
Changed lines of the file:
@@
 F 0 "J38" H 10488 5864 50  0000 L CNN
 F 1 "Conn_01x04_MountingPin" H 10488 5773 50  0000 L CNN
-F 2 "Connector_JST:JST_SH_BM04B-SRSS-TB_1x04-1MP_P1.00mm_Vertical" H 10400 5950 50  0001 C CNN
+F 2 "Connector_JST:JST_SH_SM04B-SRSS-TB_1x04-1MP_P1.00mm_Horizontal" H 10400 5950 50  0001 C CNN
 F 3 "~" H 10400 5950 50  0001 C CNN
 	1    10400 5950
@@
 F 0 "J37" H 10438 1764 50  0000 L CNN
 F 1 "Conn_01x04_MountingPin" H 10438 1673 50  0000 L CNN
-F 2 "Connector_JST:JST_SH_BM04B-SRSS-TB_1x04-1MP_P1.00mm_Vertical" H 10350 1850 50  0001 C CNN
+F 2 "Connector_JST:JST_SH_SM04B-SRSS-TB_1x04-1MP_P1.00mm_Horizontal" H 10350 1850 50  0001 C CNN
 F 3 "~" H 10350 1850 50  0001 C CNN
 	1    10350 1850
@@
 Wire Wire Line
 	4450 6650 4450 6950
+Text Label 2300 1250 0    50   ~ 0
+Q1-SDA
+Text Label 2300 950  0    50   ~ 0
+Q1-SCL
+Text Label 5200 6350 0    50   ~ 0
+Q2-SDA
+Text Label 5200 6050 0    50   ~ 0
+Q2-SCL
+Text Label 2300 1850 0    50   ~ 0
+Q1-GND
 Text Label 2300 1550 0    50   ~ 0
-Q1-SDA
-Text Label 2300 1850 0    50   ~ 0
-Q1-SCL
+Q1-3v3
+Text Label 5200 6950 0    50   ~ 0
+Q2-GND
 Text Label 5200 6650 0    50   ~ 0
-Q2-SDA
-Text Label 5200 6950 0    50   ~ 0
-Q2-SCL
-Text Label 2300 950  0    50   ~ 0
-Q1-GND
-Text Label 2300 1250 0    50   ~ 0
-Q1-3v3
-Text Label 5200 6050 0    50   ~ 0
-Q2-GND
-Text Label 5200 6350 0    50   ~ 0
 Q2-3v3
 Wire Wire Line
