File: boards/proto-quarter/proto-quarter.kicad_pcb (KiCad board)
At the start: 2 copper layers, 47 x 31 mm, 18 parts, among them J1 Conn_01x06, J10 Conn_01x10, J11 Conn_01x10, J12 Conn_01x10, J13 Conn_01x10, J14 Conn_01x10, J16 Conn_01x04, J18 Conn_01x04, J2 Conn_01x06, J3 Conn_01x10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

Commit message: Start to fix the proto board connectors.
Half board is fixed, quarter board requires reducing the length of a couple
of the connectors, namely the power rails and the top-right proto line.
Parts:
- J37, J38: footprint Connector_JST:JST_SH_BM04B-SRSS-TB_1x04-1MP_P1.00mm_Vertical -> Connector_JST:JST_SH_SM04B-SRSS-TB_1x04-1MP_P1.00mm_Horizontal
- moved J37 0.93 mm to (185.4, 87.9), turned to 180 degrees
- moved J38 0.88 mm to (209.6, 87.9), turned to 180 degrees
Routing:
- net /Q1-GND: track 63.7 -> 22.9 mm, vias 4 -> 0
- net /Q1-3v3: track 50.7 -> 22.9 mm, vias 1 -> 0
- net /Q1-SDA: track 26.8 -> 12.7 mm
- net /Q1-SCL: track 26.2 -> 12.7 mm, vias 1 -> 0
