File: boards/proto-quarter/proto-quarter.sch (KiCad schematic (older format))
At the start: 18 parts, among them J1 Conn_01x06, J10 Conn_01x10, J11 Conn_01x10, J12 Conn_01x10, J13 Conn_01x10, J14 Conn_01x10, J16 Conn_01x04, J18 Conn_01x04, J2 Conn_01x06, J3 Conn_01x10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

Commit message: Start to fix the proto board connectors.
Half board is fixed, quarter board requires reducing the length of a couple
of the connectors, namely the power rails and the top-right proto line.
Parts:
- J37, J38: footprint Connector_JST:JST_SH_BM04B-SRSS-TB_1x04-1MP_P1.00mm_Vertical -> Connector_JST:JST_SH_SM04B-SRSS-TB_1x04-1MP_P1.00mm_Horizontal
Changed lines of the file:
@@
 F 0 "J38" H 10488 5864 50  0000 L CNN
 F 1 "Conn_01x04_MountingPin" H 10488 5773 50  0000 L CNN
-F 2 "Connector_JST:JST_SH_BM04B-SRSS-TB_1x04-1MP_P1.00mm_Vertical" H 10400 5950 50  0001 C CNN
+F 2 "Connector_JST:JST_SH_SM04B-SRSS-TB_1x04-1MP_P1.00mm_Horizontal" H 10400 5950 50  0001 C CNN
 F 3 "~" H 10400 5950 50  0001 C CNN
 	1    10400 5950
@@
 F 0 "J37" H 10438 1764 50  0000 L CNN
 F 1 "Conn_01x04_MountingPin" H 10438 1673 50  0000 L CNN
-F 2 "Connector_JST:JST_SH_BM04B-SRSS-TB_1x04-1MP_P1.00mm_Vertical" H 10350 1850 50  0001 C CNN
+F 2 "Connector_JST:JST_SH_SM04B-SRSS-TB_1x04-1MP_P1.00mm_Horizontal" H 10350 1850 50  0001 C CNN
 F 3 "~" H 10350 1850 50  0001 C CNN
 	1    10350 1850
