File: boards/black-pill-breakout/black-pill-breakout.sch (KiCad schematic (older format))
At the start: 26 parts, among them J1 Conn_01x04_MountingPin, J10 Conn_01x06, J11 Conn_01x06, J12 Conn_01x06, J13 Conn_01x06, J14 Conn_01x06, J15 Conn_01x06, J16 Conn_01x06, J17 Conn_01x06, J18 Conn_01x06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

Commit message: Board Complete - Pre-Export
Parts:
- added J20: Conn_01x04, Connector_PinSocket_2.54mm:PinSocket_1x04_P2.54mm_Vertical, symbol Connector_Generic:Conn_01x04
- gave numbers to parts that had none: 2
Connections:
- net GPIO8: now also U?1.10 (A15); no longer U?1.8 (A11)
- net at U?1.38 (B0): now also J20.4 (Pin_4)
- net at U?1.39 (B1): now also J20.3 (Pin_3)
- net at U?1.40 (B2): now also J20.2 (Pin_2)
- net at U?1.41 (B10): now also J20.1 (Pin_1)
- no-connect marks 0 -> 8
Other:
- note added: "USB"
Changed lines of the file:
@@
 Text Label 2300 2800 3    50   ~ 0
 GPIO7
-Text Label 2400 2800 3    50   ~ 0
-GPIO8
 Text Label 9550 5500 2    50   ~ 0
 GPIO1
@@
 Connection ~ 9650 5700
 $Comp
-L Jumper:SolderJumper_2_Open JP?
+L Jumper:SolderJumper_2_Open JP1
 U 1 1 6083046C
 P 8450 2350
-F 0 "JP?" V 8450 2418 50  0000 L CNN
+F 0 "JP1" V 8450 2418 50  0000 L CNN
 F 1 "SolderJumper_2_Open" V 8495 2418 50  0001 L CNN
 F 2 "Jumper:SolderJumper-2_P1.3mm_Open_TrianglePad1.0x1.5mm" H 8450 2350 50  0001 C CNN
@@
 $EndComp
 $Comp
-L Jumper:SolderJumper_2_Open JP?
+L Jumper:SolderJumper_2_Open JP2
 U 1 1 6083209C
 P 8450 2650
-F 0 "JP?" V 8300 2450 50  0000 L CNN
+F 0 "JP2" V 8300 2450 50  0000 L CNN
 F 1 "SolderJumper_2_Open" V 8400 1750 50  0001 L CNN
 F 2 "Jumper:SolderJumper-2_P1.3mm_Open_TrianglePad1.0x1.5mm" H 8450 2650 50  0001 C CNN
@@
 Connection ~ 8450 2500
 $Comp
-L power:+5V #PWR?
+L power:+5V #PWR0133
 U 1 1 6086425C
 P 8450 2200
-F 0 "#PWR?" H 8450 2050 50  0001 C CNN
+F 0 "#PWR0133" H 8450 2050 50  0001 C CNN
 F 1 "+5V" H 8465 2373 50  0000 C CNN
 F 2 "" H 8450 2200 50  0001 C CNN
@@
 Wire Notes Line
 	8850 1700 8850 3150
+$Comp
+L Connector_Generic:Conn_01x04 J20
+U 1 1 608D965C
+P 2100 750
+F 0 "J20" V 2064 462 50  0000 R CNN
+F 1 "Conn_01x04" V 1973 462 50  0000 R CNN
+F 2 "Connector_PinSocket_2.54mm:PinSocket_1x04_P2.54mm_Vertical" H 2100 750 50  0001 C CNN
+F 3 "~" H 2100 750 50  0001 C CNN
+	1    2100 750
+	0    -1   -1   0
+$EndComp
+Wire Wire Line
+	2000 950  2000 1700
+Wire Wire Line
+	2100 1700 2100 950
+Wire Wire Line
+	2200 1700 2200 950
+Wire Wire Line
+	2300 950  2300 1700
+NoConn ~ 3300 1700
+NoConn ~ 3400 1700
+NoConn ~ 3500 1700
+NoConn ~ 3600 1700
+NoConn ~ 2900 2800
+NoConn ~ 2800 2800
+NoConn ~ 2500 2800
+NoConn ~ 2400 2800
+Text Notes 2400 2850 3    50   ~ 0
+USB
+Text Notes 2500 2850 3    50   ~ 0
+USB
+Text Label 2600 2800 3    50   ~ 0
+GPIO8
 $EndSCHEMATC

Commit message: Update
Other:
- moved on the sheet: J20, U?1
Changed lines of the file:
@@
 L usb-c-pill:weact-black-pill U?1
 U 1 1 603C6501
-P 1600 2250
-F 0 "U?1" V 1646 2377 50  0000 L CNN
-F 1 "weact-black-pill" V 1555 2377 50  0000 L CNN
-F 2 "usb-c-pill:weact-blackpill" H 1600 2400 50  0001 C CNN
-F 3 "" H 1600 2400 50  0001 C CNN
-	1    1600 2250
+P 1900 2800
+F 0 "U?1" V 1946 2927 50  0000 L CNN
+F 1 "weact-black-pill" V 1855 2927 50  0000 L CNN
+F 2 "usb-c-pill:weact-blackpill" H 1900 2950 50  0001 C CNN
+F 3 "" H 1900 2950 50  0001 C CNN
+	1    1900 2800
 	0    -1   -1   0
 $EndComp
@@
 L power:+5V #PWR0101
 U 1 1 6044A91F
-P 1450 1500
-F 0 "#PWR0101" H 1450 1350 50  0001 C CNN
-F 1 "+5V" V 1465 1673 50  0000 C CNN
-F 2 "" H 1450 1500 50  0001 C CNN
-F 3 "" H 1450 1500 50  0001 C CNN
-	1    1450 1500
+P 1750 2050
+F 0 "#PWR0101" H 1750 1900 50  0001 C CNN
+F 1 "+5V" V 1765 2223 50  0000 C CNN
+F 2 "" H 1750 2050 50  0001 C CNN
+F 3 "" H 1750 2050 50  0001 C CNN
+	1    1750 2050
 	0    -1   -1   0
 $EndComp
@@
 L power:GND #PWR0102
 U 1 1 6044DEE7
-P 1450 1350
-F 0 "#PWR0102" H 1450 1100 50  0001 C CNN
-F 1 "GND" V 1455 1222 50  0000 R CNN
-F 2 "" H 1450 1350 50  0001 C CNN
-F 3 "" H 1450 1350 50  0001 C CNN
-	1    1450 1350
+P 1750 1900
+F 0 "#PWR0102" H 1750 1650 50  0001 C CNN
+F 1 "GND" V 1755 1772 50  0000 R CNN
+F 2 "" H 1750 1900 50  0001 C CNN
+F 3 "" H 1750 1900 50  0001 C CNN
+	1    1750 1900
 	0    1    1    0
 $EndComp
@@
 L power:+3V3 #PWR0103
 U 1 1 6044E5C3
-P 1450 1200
-F 0 "#PWR0103" H 1450 1050 50  0001 C CNN
-F 1 "+3V3" V 1465 1328 50  0000 L CNN
-F 2 "" H 1450 1200 50  0001 C CNN
-F 3 "" H 1450 1200 50  0001 C CNN
-	1    1450 1200
+P 1750 1750
+F 0 "#PWR0103" H 1750 1600 50  0001 C CNN
+F 1 "+3V3" V 1765 1878 50  0000 L CNN
+F 2 "" H 1750 1750 50  0001 C CNN
+F 3 "" H 1750 1750 50  0001 C CNN
+	1    1750 1750
 	0    -1   -1   0
 $EndComp
 Wire Wire Line
-	1700 1700 1700 1500
-Wire Wire Line
-	1700 1500 1450 1500
-Wire Wire Line
-	1800 1700 1800 1350
-Wire Wire Line
-	1800 1350 1450 1350
-Wire Wire Line
-	1900 1700 1900 1200
-Wire Wire Line
-	1900 1200 1450 1200
+	2000 2250 2000 2050
+Wire Wire Line
+	2000 2050 1750 2050
+Wire Wire Line
+	2100 2250 2100 1900
+Wire Wire Line
+	2100 1900 1750 1900
+Wire Wire Line
+	2200 2250 2200 1750
+Wire Wire Line
+	2200 1750 1750 1750
 $Comp
 L power:+5V #PWR0104
 U 1 1 6045B305
-P 3700 3200
-F 0 "#PWR0104" H 3700 3050 50  0001 C CNN
-F 1 "+5V" V 3715 3373 50  0000 C CNN
-F 2 "" H 3700 3200 50  0001 C CNN
-F 3 "" H 3700 3200 50  0001 C CNN
-	1    3700 3200
+P 4000 3750
+F 0 "#PWR0104" H 4000 3600 50  0001 C CNN
+F 1 "+5V" V 4015 3923 50  0000 C CNN
+F 2 "" H 4000 3750 50  0001 C CNN
+F 3 "" H 4000 3750 50  0001 C CNN
+	1    4000 3750
 	0    1    -1   0
 $EndComp
@@
 L power:GND #PWR0105
 U 1 1 6045B30B
-P 3700 3050
-F 0 "#PWR0105" H 3700 2800 50  0001 C CNN
-F 1 "GND" V 3705 2922 50  0000 R CNN
-F 2 "" H 3700 3050 50  0001 C CNN
-F 3 "" H 3700 3050 50  0001 C CNN
-	1    3700 3050
+P 4000 3600
+F 0 "#PWR0105" H 4000 3350 50  0001 C CNN
+F 1 "GND" V 4005 3472 50  0000 R CNN
+F 2 "" H 4000 3600 50  0001 C CNN
+F 3 "" H 4000 3600 50  0001 C CNN
+	1    4000 3600
 	0    -1   1    0
 $EndComp
 Wire Wire Line
-	3600 2800 3600 2900
-Wire Wire Line
-	3600 2900 3700 2900
-Wire Wire Line
-	3500 2800 3500 3050
-Wire Wire Line
-	3500 3050 3700 3050
-Wire Wire Line
-	3400 2800 3400 3200
-Wire Wire Line
-	3400 3200 3700 3200
+	3900 3350 3900 3450
+Wire Wire Line
+	3900 3450 4000 3450
+Wire Wire Line
+	3800 3350 3800 3600
+Wire Wire Line
+	3800 3600 4000 3600
+Wire Wire Line
+	3700 3350 3700 3750
+Wire Wire Line
+	3700 3750 4000 3750
 $Comp
 L power:GND #PWR0106
 U 1 1 6046DF1A
-P 3750 2100
-F 0 "#PWR0106" H 3750 1850 50  0001 C CNN
-F 1 "GND" V 3755 1972 50  0000 R CNN
-F 2 "" H 3750 2100 50  0001 C CNN
-F 3 "" H 3750 2100 50  0001 C CNN
-	1    3750 2100
+P 4050 2650
+F 0 "#PWR0106" H 4050 2400 50  0001 C CNN
+F 1 "GND" V 4055 2522 50  0000 R CNN
+F 2 "" H 4050 2650 50  0001 C CNN
+F 3 "" H 4050 2650 50  0001 C CNN
+	1    4050 2650
 	0    -1   1    0
 $EndComp
@@
 L power:+3V3 #PWR0107
 U 1 1 604750A8
-P 3700 2900
-F 0 "#PWR0107" H 3700 2750 50  0001 C CNN
-F 1 "+3V3" V 3715 3028 50  0000 L CNN
-F 2 "" H 3700 2900 50  0001 C CNN
-F 3 "" H 3700 2900 50  0001 C CNN
-	1    3700 2900
+P 4000 3450
+F 0 "#PWR0107" H 4000 3300 50  0001 C CNN
+F 1 "+3V3" V 4015 3578 50  0000 L CNN
+F 2 "" H 4000 3450 50  0001 C CNN
+F 3 "" H 4000 3450 50  0001 C CNN
+	1    4000 3450
 	0    1    -1   0
 $EndComp
@@
 L power:+3V3 #PWR0108
 U 1 1 60477BBB
-P 3750 2400
-F 0 "#PWR0108" H 3750 2250 50  0001 C CNN
-F 1 "+3V3" V 3765 2528 50  0000 L CNN
-F 2 "" H 3750 2400 50  0001 C CNN
-F 3 "" H 3750 2400 50  0001 C CNN
-	1    3750 2400
+P 4050 2950
+F 0 "#PWR0108" H 4050 2800 50  0001 C CNN
+F 1 "+3V3" V 4065 3078 50  0000 L CNN
+F 2 "" H 4050 2950 50  0001 C CNN
+F 3 "" H 4050 2950 50  0001 C CNN
+	1    4050 2950
 	0    1    -1   0
 $EndComp
-Text Label 3750 2200 0    50   ~ 0
+Text Label 4050 2750 0    50   ~ 0
 SWCLK
-Text Label 3750 2300 0    50   ~ 0
+Text Label 4050 2850 0    50   ~ 0
 SWDIO
-Text Label 3000 2800 3    50   ~ 0
+Text Label 3300 3350 3    50   ~ 0
 I2C-SCL
-Text Label 3100 2800 3    50   ~ 0
+Text Label 3400 3350 3    50   ~ 0
 I2C-SDA
-Text Label 2400 1700 1    50   ~ 0
+Text Label 2700 2250 1    50   ~ 0
 SPI-COPI
-Text Label 2500 1700 1    50   ~ 0
+Text Label 2800 2250 1    50   ~ 0
 SPI-CIPO
-Text Label 2600 1700 1    50   ~ 0
+Text Label 2900 2250 1    50   ~ 0
 SPI-SCK
-Text Label 2700 1700 1    50   ~ 0
+Text Label 3000 2250 1    50   ~ 0
 ~SPI-CS
-Text Label 2800 1700 1    50   ~ 0
+Text Label 3100 2250 1    50   ~ 0
 USART-RX
-Text Label 2900 1700 1    50   ~ 0
+Text Label 3200 2250 1    50   ~ 0
 USART-TX
-Text Label 3000 1700 1    50   ~ 0
+Text Label 3300 2250 1    50   ~ 0
 USART-RTS
-Text Label 3100 1700 1    50   ~ 0
+Text Label 3400 2250 1    50   ~ 0
 USART-CTS
-Text Label 3200 1700 1    50   ~ 0
+Text Label 3500 2250 1    50   ~ 0
 ~SWD-RST
 $Comp
@@
 Text Label 7850 2100 0    50   ~ 0
 ~SWD-RST
-Text Label 2700 2800 3    50   ~ 0
+Text Label 3000 3350 3    50   ~ 0
 SWO
 $Comp
@@
 Wire Wire Line
 	8000 3950 8000 3850
-Text Label 3300 2800 3    50   ~ 0
+Text Label 3600 3350 3    50   ~ 0
 ~I2C-INT
-Text Label 3200 2800 3    50   ~ 0
+Text Label 3500 3350 3    50   ~ 0
 ~I2C-RST
 Text Notes 9100 5150 0    50   ~ 0
@@
 	0    1    1    0
 $EndComp
-Text Label 1700 2800 3    50   ~ 0
+Text Label 2000 3350 3    50   ~ 0
 GPIO1
-Text Label 1800 2800 3    50   ~ 0
+Text Label 2100 3350 3    50   ~ 0
 GPIO2
-Text Label 1900 2800 3    50   ~ 0
+Text Label 2200 3350 3    50   ~ 0
 GPIO3
-Text Label 2000 2800 3    50   ~ 0
+Text Label 2300 3350 3    50   ~ 0
 GPIO4
-Text Label 2100 2800 3    50   ~ 0
+Text Label 2400 3350 3    50   ~ 0
 GPIO5
-Text Label 2200 2800 3    50   ~ 0
+Text Label 2500 3350 3    50   ~ 0
 GPIO6
-Text Label 2300 2800 3    50   ~ 0
+Text Label 2600 3350 3    50   ~ 0
 GPIO7
 Text Label 9550 5500 2    50   ~ 0
@@
 L Connector_Generic:Conn_01x04 J20
 U 1 1 608D965C
-P 2100 750
-F 0 "J20" V 2064 462 50  0000 R CNN
-F 1 "Conn_01x04" V 1973 462 50  0000 R CNN
-F 2 "Connector_PinSocket_2.54mm:PinSocket_1x04_P2.54mm_Vertical" H 2100 750 50  0001 C CNN
-F 3 "~" H 2100 750 50  0001 C CNN
-	1    2100 750
+P 2400 1300
+F 0 "J20" V 2364 1012 50  0000 R CNN
+F 1 "Conn_01x04" V 2273 1012 50  0000 R CNN
+F 2 "Connector_PinSocket_2.54mm:PinSocket_1x04_P2.54mm_Vertical" H 2400 1300 50  0001 C CNN
+F 3 "~" H 2400 1300 50  0001 C CNN
+	1    2400 1300
 	0    -1   -1   0
 $EndComp
 Wire Wire Line
-	2000 950  2000 1700
-Wire Wire Line
-	2100 1700 2100 950
-Wire Wire Line
-	2200 1700 2200 950
-Wire Wire Line
-	2300 950  2300 1700
-NoConn ~ 3300 1700
-NoConn ~ 3400 1700
-NoConn ~ 3500 1700
-NoConn ~ 3600 1700
-NoConn ~ 2900 2800
-NoConn ~ 2800 2800
-NoConn ~ 2500 2800
-NoConn ~ 2400 2800
-Text Notes 2400 2850 3    50   ~ 0
+	2300 1500 2300 2250
+Wire Wire Line
+	2400 2250 2400 1500
+Wire Wire Line
+	2500 2250 2500 1500
+Wire Wire Line
+	2600 1500 2600 2250
+NoConn ~ 3600 2250
+NoConn ~ 3700 2250
+NoConn ~ 3800 2250
+NoConn ~ 3900 2250
+NoConn ~ 3200 3350
+NoConn ~ 3100 3350
+NoConn ~ 2800 3350
+NoConn ~ 2700 3350
+Text Notes 2700 3400 3    50   ~ 0
 USB
-Text Notes 2500 2850 3    50   ~ 0
+Text Notes 2800 3400 3    50   ~ 0
 USB
-Text Label 2600 2800 3    50   ~ 0
+Text Label 2900 3350 3    50   ~ 0
 GPIO8
 $EndSCHEMATC
