File: boards/sprocket/_autosave-sprocket.sch (KiCad schematic (older format))
At the start: 39 parts, among them J4 Conn_01x04_MountingPin, J5 Conn_01x04_MountingPin, J6 Conn_01x04_MountingPin, J7 Conn_01x04_MountingPin, Q1 NX7002BKR, SW1 SW_Push, SW2 SW_Push, U1 STM32G031G8U6, U2 AP2210N-3.3TRG1

Commit message: Work
Parts:
- J1: renamed from J?; footprint (none) -> Everything:sprocket-pins
Changed lines of the file:
@@
 Circuit Components
 $Comp
-L Everything:SPROCKET-CONN J?
+L Everything:SPROCKET-CONN J1
 U 1 1 607795BD
 P 1400 5350
-F 0 "J?" H 1400 5515 50  0000 C CNN
+F 0 "J1" H 1400 5515 50  0000 C CNN
 F 1 "SPROCKET-CONN" H 1400 5424 50  0000 C CNN
-F 2 "" H 1400 5400 50  0001 C CNN
+F 2 "Everything:sprocket-pins" H 1400 5400 50  0001 C CNN
 F 3 "" H 1400 5400 50  0001 C CNN
 	1    1400 5350

Commit message: About to give up again
Parts:
- removed JP1, JP2, JP5, JP6: SolderJumper_2_Open, Jumper:SolderJumper-2_P1.3mm_Open_TrianglePad1.0x1.5mm, symbol Jumper:SolderJumper_2_Open
- removed R1: 10K, Resistor_SMD:R_0402_1005Metric, symbol Device:R
- JP3, JP4: footprint Jumper:SolderJumper-2_P1.3mm_Open_TrianglePad1.0x1.5mm -> Jumper:SolderJumper-2_P1.3mm_Open_RoundedPad1.0x1.5mm
Connections:
- net QWIIC2-SCL is gone; now on net I2C2-SCL: J6.4 (Pin_4), J7.4 (Pin_4), JP4.2 (B)
- net I2C1-SDA: now also JP3.2 (B); no longer JP3.1 (A)
- net I2C2-SDA: now also J6.3 (Pin_3), J7.3 (Pin_3), JP3.1 (A)
- removed net QWIIC2-SDA: J6.3 (Pin_3), J7.3 (Pin_3), JP3.2 (B)
Other:
- note removed: "I2C2 to QWIIC Jumpers"
- note removed: "Open Drain UART Jumper"
- note removed: "Open Drain UART Pullup\n"
Changed lines of the file:
@@
 F 0 "JP3" H 1350 4705 50  0000 C CNN
 F 1 "SolderJumper_2_Open" H 1350 4614 50  0000 C CNN
-F 2 "Jumper:SolderJumper-2_P1.3mm_Open_TrianglePad1.0x1.5mm" H 1350 4500 50  0001 C CNN
+F 2 "Jumper:SolderJumper-2_P1.3mm_Open_RoundedPad1.0x1.5mm" H 1350 4500 50  0001 C CNN
 F 3 "~" H 1350 4500 50  0001 C CNN
 	1    1350 4500
-	1    0    0    -1
+	-1   0    0    -1
 $EndComp
 $Comp
@@
 F 0 "JP4" H 1350 5055 50  0000 C CNN
 F 1 "SolderJumper_2_Open" H 1350 4964 50  0000 C CNN
-F 2 "Jumper:SolderJumper-2_P1.3mm_Open_TrianglePad1.0x1.5mm" H 1350 4850 50  0001 C CNN
+F 2 "Jumper:SolderJumper-2_P1.3mm_Open_RoundedPad1.0x1.5mm" H 1350 4850 50  0001 C CNN
 F 3 "~" H 1350 4850 50  0001 C CNN
 	1    1350 4850
@@
 Text Notes 1600 4200 2    50   ~ 0
 QWIIC Daisy Chain Jumpers
-$Comp
-L Jumper:SolderJumper_2_Open JP6
-U 1 1 6067FFF6
-P 3100 4850
-F 0 "JP6" H 3100 5055 50  0000 C CNN
-F 1 "SolderJumper_2_Open" H 3100 4964 50  0000 C CNN
-F 2 "Jumper:SolderJumper-2_P1.3mm_Open_TrianglePad1.0x1.5mm" H 3100 4850 50  0001 C CNN
-F 3 "~" H 3100 4850 50  0001 C CNN
-	1    3100 4850
-	1    0    0    -1
-$EndComp
-Text Label 2950 4850 2    50   ~ 0
-QWIIC2-SDA
-Text Label 3250 4850 0    50   ~ 0
-QWIIC2-SCL
-Text Notes 3450 4600 2    50   ~ 0
-Open Drain UART Jumper
-$Comp
-L Jumper:SolderJumper_2_Open JP5
-U 1 1 6069AF59
-P 3100 4300
-F 0 "JP5" H 3100 4505 50  0000 C CNN
-F 1 "SolderJumper_2_Open" H 3100 4414 50  0000 C CNN
-F 2 "Jumper:SolderJumper-2_P1.3mm_Open_TrianglePad1.0x1.5mm" H 3100 4300 50  0001 C CNN
-F 3 "~" H 3100 4300 50  0001 C CNN
-	1    3100 4300
-	1    0    0    -1
-$EndComp
-$Comp
-L Device:R R1
-U 1 1 606A0041
-P 3400 4300
-F 0 "R1" V 3300 4300 50  0000 C CNN
-F 1 "10K" V 3400 4300 50  0000 C CNN
-F 2 "Resistor_SMD:R_0402_1005Metric" V 3330 4300 50  0001 C CNN
-F 3 "~" H 3400 4300 50  0001 C CNN
-	1    3400 4300
-	0    -1   -1   0
-$EndComp
-$Comp
-L power:+3V3 #PWR0135
-U 1 1 606A1D31
-P 3550 4300
-F 0 "#PWR0135" H 3550 4150 50  0001 C CNN
-F 1 "+3V3" H 3565 4473 50  0000 C CNN
-F 2 "" H 3550 4300 50  0001 C CNN
-F 3 "" H 3550 4300 50  0001 C CNN
-	1    3550 4300
-	1    0    0    -1
-$EndComp
-Text Label 2950 4300 2    50   ~ 0
-QWIIC2-SCL
-Text Notes 3400 4000 2    50   ~ 0
-Open Drain UART Pullup\n
 Wire Notes Line
 	3900 3850 2300 3850
@@
 Text Label 1500 2950 0    50   ~ 0
 I2C1-SDA
-$Comp
-L Jumper:SolderJumper_2_Open JP1
-U 1 1 606C75BE
-P 1350 3600
-F 0 "JP1" H 1350 3805 50  0000 C CNN
-F 1 "SolderJumper_2_Open" H 1350 3714 50  0000 C CNN
-F 2 "Jumper:SolderJumper-2_P1.3mm_Open_TrianglePad1.0x1.5mm" H 1350 3600 50  0001 C CNN
-F 3 "~" H 1350 3600 50  0001 C CNN
-	1    1350 3600
-	1    0    0    -1
-$EndComp
-$Comp
-L Jumper:SolderJumper_2_Open JP2
-U 1 1 606C75C4
-P 1350 3950
-F 0 "JP2" H 1350 4155 50  0000 C CNN
-F 1 "SolderJumper_2_Open" H 1350 4064 50  0000 C CNN
-F 2 "Jumper:SolderJumper-2_P1.3mm_Open_TrianglePad1.0x1.5mm" H 1350 3950 50  0001 C CNN
-F 3 "~" H 1350 3950 50  0001 C CNN
-	1    1350 3950
-	1    0    0    -1
-$EndComp
-Text Label 1500 3600 0    50   ~ 0
+Text Label 1200 3250 2    50   ~ 0
 QWIIC2-SDA
-Text Label 1500 3950 0    50   ~ 0
+Text Label 1200 3400 2    50   ~ 0
 QWIIC2-SCL
-Text Label 1200 3600 2    50   ~ 0
+Text Label 1500 3250 0    50   ~ 0
 I2C2-SDA
-Text Label 1200 3950 2    50   ~ 0
+Text Label 1500 3400 0    50   ~ 0
 I2C2-SCL
 Wire Wire Line
@@
 	1200 3100 1500 3100
 Wire Notes Line
-	500  3250 2300 3250
-Wire Notes Line
 	2300 2650 2300 7750
-Text Notes 1450 3350 2    50   ~ 0
-I2C2 to QWIIC Jumpers
 Text Notes 1750 2750 2    50   ~ 0
 Unnecessary Labels for Clarity
@@
 Text Label 1950 7050 0    50   ~ 0
 UART-TX
-Wire Notes Line
-	2350 4450 3850 4450
 $Comp
 L Connector_Generic:Conn_01x02 MH1
@@
 	1    0    0    -1
 $EndComp
+Wire Wire Line
+	1500 3250 1200 3250
+Wire Wire Line
+	1500 3400 1200 3400
 $EndSCHEMATC
