File: boards/sprocket/sprocket-panel.kicad_pcb (KiCad board)
At the start: 4 copper layers, 97 x 87 mm, 494 parts, among them J1 SPROCKET-CONN, J4 Conn_01x04_MountingPin, J5 Conn_01x04_MountingPin, J6 Conn_01x04_MountingPin, J7 Conn_01x04_MountingPin, Q1 NX7002BKR, SW1 SW_Push, SW2 SW_Push, U1 STM32G031G8U6, U2 AP2210N-3.3TRG1

Commit message: Add recent projects
Other:
- board text added: "!"
- board text added: "*"
- board text added: "1 spi, swd"
- board text added: "1 uart, 2 i2c,"
- board text added: "28"
- board text added: "3v3, 5v ok"
- board text added: "64 mhz"
- board text added: "64k flash"
- board text added: "6x adc +"
- board text added: "7x"
- board text added: "8 gpios:"
- board text added: "8k"
- board text added: "8x"
- board text added: "8x pwm"
- board text added: "buy it, use it, break it, fix it,"
- board text added: "call it, find it, view it, code it,"
- board text added: "hello!"
- board text added: "jam unlock it. technologic."
- board text added: "pins"
- board text added: "ram"
- board text added: "trash it, change it, mail"
- board text added: "upgrade it. lock it, fill it,"
- board text removed: "7"
- board text removed: "8"
- board text removed: "funky!"
- board text removed: "get"
- board text removed: "never stop."

Commit message: putzing
Routing:
- net Board_4-+3V3: track 51.3 -> 50.5 mm
- net Board_3-+3V3: track 51.3 -> 50.5 mm
- net Board_5-+3V3: track 51.3 -> 50.5 mm
- net Board_8-+3V3: track 51.3 -> 50.5 mm
- net Board_7-+3V3: track 51.3 -> 50.5 mm
- net Board_6-+3V3: track 51.3 -> 50.5 mm
- net Board_9-+3V3: track 51.3 -> 50.5 mm
- net Board_2-+3V3: track 51.3 -> 50.5 mm
- net Board_10-+3V3: track 51.3 -> 50.5 mm
- net Board_1-+3V3: track 51.3 -> 50.5 mm
- net Board_4-GND: track 57.3 -> 56.7 mm
- net Board_3-GND: track 57.3 -> 56.7 mm
- net Board_9-GND: track 57.3 -> 56.7 mm
- net Board_8-GND: track 57.3 -> 56.7 mm
- net Board_7-GND: track 57.3 -> 56.7 mm
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