File: boards/sprocket/sprocket.kicad_pcb (KiCad board)
At the start: 4 copper layers, 47 x 15 mm, 34 parts, among them J1 SPROCKET-CONN, J4 Conn_01x04_MountingPin, J5 Conn_01x04_MountingPin, J6 Conn_01x04_MountingPin, J7 Conn_01x04_MountingPin, Q1 NX7002BKR, SW1 SW_Push, SW2 SW_Push, U1 STM32G031G8U6, U2 AP2210N-3.3TRG1

Commit message: Pre-order
Parts:
- added TP1: TestPoint, TestPoint:TestPoint_Pad_D1.5mm, F.Cu at (107.5, 89.3)
- moved R5 0.30 mm to (114.2, 82.2)
Routing:
- net /SMARTLED-OUT: track 0.00 -> 11.3 mm, vias 0 -> 2
- net +3V3: track 54.1 -> 51.3 mm, vias 7 -> 8
- added copper zone on F.Cu, net +3V3
Other:
- board text added: "'21"
- board text added: "1"
- board text added: "2"
- board text added: "3"
- board text added: "3v3"
- board text added: "4"
- board text added: "5"
- board text added: "5V0"
- board text added: "5v0"
- board text added: "6"
- board text added: "7"
- board text added: "8"
- board text added: "@bitshiftmask"
- board text added: "GND"
- board text added: "beep"
- board text added: "blink"
- board text added: "boop"
- board text added: "build tools"
- board text added: "chain"
- board text added: "cipo"
- board text added: "clack"
- board text added: "clank"
- board text added: "click"
- board text added: "clink"
- board text added: "clk"
- board text added: "copi"
- board text added: "csn"
- board text added: "daisy"
- board text added: "dio"
- board text added: "drop"
- board text added: "fidget"
- board text added: "funky!"
- board text added: "get"
- board text added: "gnd"
- board text added: "i2c1"
- board text added: "i2c2"
- board text added: "ldo"
- board text added: "led"
- board text added: "lvl"
- board text added: "march"
- board text added: "never stop."
- board text added: "nrst"
- board text added: "pause"
- board text added: "pow"
- board text added: "qwiic"
- board text added: "rattle"
- board text added: "roll"
- board text added: "rx"
- board text added: "sck"
- board text added: "scl"
- board text added: "sda"
- board text added: "shake"
- board text added: "shift"
- board text added: "shine"
- board text added: "smart"
- board text added: "sprocket!"
- board text added: "stm32g0"
- board text added: "swirl"
- board text added: "tell stories"
- board text added: "think"
- board text added: "tx"

Commit message: Pre-export
Other:
- board text added: "!"
- board text added: "*"
- board text added: "1 spi, swd"
- board text added: "1 uart, 2 i2c,"
- board text added: "28"
- board text added: "3v3, 5v ok"
- board text added: "64 mhz"
- board text added: "64k flash"
- board text added: "6x adc +"
- board text added: "7x"
- board text added: "8 gpios:"
- board text added: "8k"
- board text added: "8x"
- board text added: "8x pwm"
- board text added: "buy it, use it, break it, fix it,"
- board text added: "call it, find it, view it, code it,"
- board text added: "hello!"
- board text added: "jam unlock it. technologic."
- board text added: "pins"
- board text added: "ram"
- board text added: "trash it, change it, mail"
- board text added: "upgrade it. lock it, fill it,"
- board text removed: "7"
- board text removed: "8"
- board text removed: "funky!"
- board text removed: "get"
- board text removed: "never stop."

Commit message: Add recent projects
Routing:
- net +3V3: track 51.3 -> 50.5 mm
- net GND: track 57.3 -> 56.7 mm
